File: VNA.sch (KiCad schematic (older format))
At the start: 4 parts

Commit message: Annoatated Schematics
Parts:
- gave numbers to parts that had none: 4
Changed lines of the file:
@@
 $EndSheet
 $Comp
-L Connector:Conn_Coaxial J?
+L Connector:Conn_Coaxial J1
 U 1 1 5B49CA40
 P 9300 1100
-F 0 "J?" H 9399 1076 50  0000 L CNN
+F 0 "J1" H 9399 1076 50  0000 L CNN
 F 1 "Conn_Coaxial" H 9399 985 50  0000 L CNN
 F 2 "Connector_Coaxial:SMA_Amphenol_132289_EdgeMount" H 9300 1100 50  0001 C CNN
@@
 $EndComp
 $Comp
-L Connector:Conn_Coaxial J?
+L Connector:Conn_Coaxial J2
 U 1 1 5B49CA81
 P 9300 1600
-F 0 "J?" H 9399 1576 50  0000 L CNN
+F 0 "J2" H 9399 1576 50  0000 L CNN
 F 1 "Conn_Coaxial" H 9399 1485 50  0000 L CNN
 F 2 "Connector_Coaxial:SMA_Amphenol_132289_EdgeMount" H 9300 1600 50  0001 C CNN
@@
 $EndComp
 $Comp
-L Connector:Conn_Coaxial J?
+L Connector:Conn_Coaxial J3
 U 1 1 5B49CB29
 P 9300 2100
-F 0 "J?" H 9399 2076 50  0000 L CNN
+F 0 "J3" H 9399 2076 50  0000 L CNN
 F 1 "Conn_Coaxial" H 9399 1985 50  0000 L CNN
 F 2 "Connector_Coaxial:SMA_Amphenol_132289_EdgeMount" H 9300 2100 50  0001 C CNN
@@
 $EndComp
 $Comp
-L Connector:Conn_Coaxial J?
+L Connector:Conn_Coaxial J4
 U 1 1 5B49CB72
 P 9300 2600
-F 0 "J?" H 9399 2576 50  0000 L CNN
+F 0 "J4" H 9399 2576 50  0000 L CNN
 F 1 "Conn_Coaxial" H 9399 2485 50  0000 L CNN
 F 2 "Connector_Coaxial:SMA_Amphenol_132289_EdgeMount" H 9300 2600 50  0001 C CNN
@@
 	7000 1250 7400 1250
 $Comp
-L power:GNDA #PWR?
+L power:GNDA #PWR075
 U 1 1 5B49E872
 P 9300 1300
-F 0 "#PWR?" H 9300 1050 50  0001 C CNN
+F 0 "#PWR075" H 9300 1050 50  0001 C CNN
 F 1 "GNDA" H 9305 1127 50  0000 C CNN
 F 2 "" H 9300 1300 50  0001 C CNN
@@
 $EndComp
 $Comp
-L power:GNDA #PWR?
+L power:GNDA #PWR076
 U 1 1 5B49E8A0
 P 9300 1800
-F 0 "#PWR?" H 9300 1550 50  0001 C CNN
+F 0 "#PWR076" H 9300 1550 50  0001 C CNN
 F 1 "GNDA" H 9305 1627 50  0000 C CNN
 F 2 "" H 9300 1800 50  0001 C CNN
@@
 $EndComp
 $Comp
-L power:GNDA #PWR?
+L power:GNDA #PWR077
 U 1 1 5B49E8CE
 P 9300 2300
-F 0 "#PWR?" H 9300 2050 50  0001 C CNN
+F 0 "#PWR077" H 9300 2050 50  0001 C CNN
 F 1 "GNDA" H 9305 2127 50  0000 C CNN
 F 2 "" H 9300 2300 50  0001 C CNN
@@
 $EndComp
 $Comp
-L power:GNDA #PWR?
+L power:GNDA #PWR078
 U 1 1 5B49E8FC
 P 9300 2800
-F 0 "#PWR?" H 9300 2550 50  0001 C CNN
+F 0 "#PWR078" H 9300 2550 50  0001 C CNN
 F 1 "GNDA" H 9305 2627 50  0000 C CNN
 F 2 "" H 9300 2800 50  0001 C CNN
